Commit message: added complete gripper model and tested with rviz

File: gripper_description/xacro/two_finger.urdf (robot description, URDF)
Before this commit: robot None, 0 links, 0 joints
Links:
- added link base, mass 9.60074e-05; visual mesh filename=package://two_finger/meshes/Base.stl scale=1 1 1
- added link block, mass 1.56518e-06; visual mesh filename=package://two_finger/meshes/Block.stl scale=1 1 1
- added link block_1, mass 1.56518e-06; visual mesh filename=package://two_finger/meshes/Block.stl scale=1 1 1
- added link block_2, mass 1.56518e-06; visual mesh filename=package://two_finger/meshes/Block.stl scale=1 1 1
- added link block_3, mass 1.56518e-06; visual mesh filename=package://two_finger/meshes/Block.stl scale=1 1 1
- added link clamp, mass 2.4104e-05; visual mesh filename=package://two_finger/meshes/Clamp.stl scale=1 1 1
- added link dynamixel_xm430_w350_r, mass 4.41073e-05; visual mesh filename=package://two_finger/meshes/dynamixel_XM430_W350_R.stl scale=1 1 1
- added link gipper_case, mass 2.86395e-05; visual mesh filename=package://two_finger/meshes/Gipper_case.stl scale=1 1 1
- added link gipper_case_1, mass 2.86395e-05; visual mesh filename=package://two_finger/meshes/Gipper_case.stl scale=1 1 1
- added link gripper_support, mass 1.89595e-05; visual mesh filename=package://two_finger/meshes/Gripper_support.stl scale=1 1 1
- added link gripper_support_1, mass 1.89595e-05; visual mesh filename=package://two_finger/meshes/Gripper_support.stl scale=1 1 1
- added link link, mass 3.47229e-06; visual mesh filename=package://two_finger/meshes/Link.stl scale=1 1 1
- added link link_1, mass 3.47229e-06; visual mesh filename=package://two_finger/meshes/Link.stl scale=1 1 1
- added link link__1__loop_closure, mass 1e-09
- added link link__2__loop_closure, mass 1e-09
- added link mgnr09r315hm, mass 7.10975e-06; visual mesh filename=package://two_finger/meshes/MGNR09R315HM.stl scale=1 1 1
- added link mgnr09r315hm_1, mass 7.10975e-06; visual mesh filename=package://two_finger/meshes/MGNR09R315HM.stl scale=1 1 1
- added link planar_4
- added link planar_4_1
- added link planar_5
- added link planar_5_1
- added link root
- added link small_motor_mount, mass 1.0786e-05; visual mesh filename=package://two_finger/meshes/Small_motor_mount.stl scale=1 1 1
- added link small_motor_test_2_base, mass 4.70869e-05; visual mesh filename=package://two_finger/meshes/Small_Motor_test_2_Base.stl scale=1 1 1
- added link soft_gripper_finger, mass 4.70738e-05; visual mesh filename=package://two_finger/meshes/soft_gripper_finger.stl scale=1 1 1
- added link soft_gripper_finger_1, mass 4.70738e-05; visual mesh filename=package://two_finger/meshes/soft_gripper_finger.stl scale=1 1 1
Joints:
- added joint fastened_1: type fixed, parent root, child clamp, origin xyz=3.46945e-18 6.93889e-18 4.33681e-18 rpy=2.13568e-32 5.31737e-33 -1.5708, axis 0 0 1
- added joint fastened_10: type fixed, parent gripper_support_1, child gipper_case_1, origin xyz=0.0085 -0.018885 0.0282 rpy=1.5708 -8.04912e-16 3.14159, axis 0 -1 0
- added joint fastened_11: type fixed, parent base, child small_motor_test_2_base, origin xyz=0.0858995 0.0065 0.0273995 rpy=-1.5708 -3.37038e-32 -1.3886e-31, axis 0 -1 0
- added joint fastened_12: type fixed, parent base, child dynamixel_xm430_w350_r, origin xyz=-0.0182005 0.04185 0.0213995 rpy=1.5708 -3.38813e-21 3.14159, axis 0 0 1
- added joint fastened_13: type fixed, parent gipper_case_1, child soft_gripper_finger, origin xyz=0.0289911 -0.0021 -0.0217317 rpy=-1.5708 2.46733e-30 -3.29899e-29, axis 0 0 -1
- added joint fastened_14: type fixed, parent gipper_case, child soft_gripper_finger_1, origin xyz=0.0289911 -0.0021 -0.0217317 rpy=-1.5708 -7.02888e-17 -7.02888e-17, axis 0 0 1
- added joint fastened_2: type fixed, parent clamp, child base, origin xyz=0.0275 -0.00989949 0.027421 rpy=-1.44607e-16 -2.00374e-16 1.5708, axis 1.73472e-16 -1 -2.00618e-32
- added joint fastened_3: type fixed, parent gripper_support, child block_1, origin xyz=-0.0131198 -0.007 -0.0121 rpy=4.74207e-19 -1.38778e-16 -4.80745e-31, axis 0 -1 0
- added joint fastened_4: type fixed, parent gripper_support, child block_3, origin xyz=-0.0131198 -0.007 0.0381 rpy=6.13299e-17 -2.498e-16 -5.19187e-31, axis 0 -1 0
- added joint fastened_5: type fixed, parent gripper_support_1, child block_2, origin xyz=-0.005 -0.00588499 -0.0121 rpy=3.14159 -1.38778e-16 -3.14159, axis 0 -1 0
- added joint fastened_6: type fixed, parent small_motor_test_2_base, child mgnr09r315hm_1, origin xyz=-0.146 -0.031 0.0035 rpy=-8.29972e-17 2.77556e-17 2.75156e-17, axis 0 1 0
- added joint fastened_7: type fixed, parent small_motor_test_2_base, child mgnr09r315hm, origin xyz=-0.146 -0.031 0.0385 rpy=-1.50861e-16 -2.498e-16 -1.44023e-16, axis 0 -1 0
- added joint fastened_8: type fixed, parent gripper_support_1, child block, origin xyz=-0.005 -0.00588499 0.0381 rpy=3.14159 8.32667e-17 3.14159, axis 0 -1 0
- added joint fastened_9: type fixed, parent gripper_support, child gipper_case, origin xyz=0.000380163 -0.02 0.0282 rpy=1.5708 -7.21645e-16 -3.14159, axis 0 -1 0
- added joint planar_4: type prismatic, parent mgnr09r315hm, child planar_4_1, origin xyz=0.129112 -0.00361501 -0.0045 rpy=-3.14159 -2.77556e-17 -3.14159, axis -1 0 0, limit lower=-10000 upper=10000 effort=1 velocity=1
- added joint planar_4_1: type prismatic, parent planar_4_1, child planar_4, origin xyz=0 0 0 rpy=0 -0 0, axis 0 -1 0, limit lower=-10000 upper=10000 effort=1 velocity=1
- added joint planar_4_2: type continuous, parent planar_4, child gripper_support_1, origin xyz=0 0 0 rpy=0 -0 0, axis 0 0 1
- added joint planar_5: type prismatic, parent mgnr09r315hm_1, child planar_5_1, origin xyz=0.0189804 -0.0025 0.0045 rpy=1.91119e-16 -5.55112e-17 -7.01768e-17, axis 1 0 0, limit lower=-10000 upper=10000 effort=1 velocity=1
- added joint planar_5_1: type prismatic, parent planar_5_1, child planar_5, origin xyz=0 0 0 rpy=0 -0 0, axis 0 1 0, limit lower=-10000 upper=10000 effort=1 velocity=1
- added joint planar_5_2: type continuous, parent planar_5, child gripper_support, origin xyz=0 0 0 rpy=0 -0 0, axis 0 0 1
- added joint revolute_1: type continuous, parent dynamixel_xm430_w350_r, child small_motor_mount, origin xyz=-0.0281 0.0135 -0.0143 rpy=-2.02118e-16 -0.349418 3.14159, axis 0 1 0
- added joint revolute_2: type continuous, parent small_motor_mount, child link_1, origin xyz=0.027 -0.009 8.42967e-18 rpy=3.14159 -0.618169 -3.14159, axis 0 -1 0
- added joint revolute_3: type continuous, parent small_motor_mount, child link, origin xyz=-0.027 -0.009 -1.93259e-17 rpy=7.33602e-17 0.615207 2.98888e-16, axis 0 -1 0
- added joint revolute_5_loop_closure: type continuous, parent gripper_support_1, child link__1__loop_closure, origin xyz=2.77556e-17 0.00811501 0.013 rpy=-7.62939e-16 0.268751 -2.48014e-16, axis 0 1 0
- added joint revolute_6_loop_closure: type continuous, parent gripper_support, child link__2__loop_closure, origin xyz=-0.00811984 0.007 0.013 rpy=-2.37866e-16 0.265789 4.03328e-17, axis 0 1 0
