Commit message: tested and calibrated the simulation gripper with physical one

File: gripper_description/xacro/two-finger-gripper.urdf.xacro (robot description, xacro)
@@ -1,487 +1,431 @@
 <?xml version="1.0"?>
 <robot xmlns:xacro="http://www.ros.org/wiki/xacro">
-  <xacro:macro name="two_finger_gripper" params="parent prefix:='' xyz:='0 0 0' rpy:='0 0 0'">
-    <joint name="${prefix}gripper_parent_to_root" type="fixed">
-      <parent link="${parent}" />
-      <child link="${prefix}gripper_root" />
-      <origin xyz="${xyz}" rpy="${rpy}" />
-    </joint>
-    <link name="${prefix}gripper_base">
-            <inertial>
-            <mass value="9.60074e-05" />
-            <origin xyz="0.00989949 0.0275 0.013491" rpy="0 -0 0" />
-            <inertia ixx="4.52785e-08" ixy="0" ixz="0" iyy="1.33505e-07" iyz="0" izz="1.57011e-07" />
-        </inertial>
-            <visual>
-            <origin xyz="-0.0701005 0.0525 0.0273995" rpy="0 -0 0" />
-            <geometry>
-                <mesh filename="package://gripper_description/meshes/soft-two-finger-gripper/Base.stl" scale="1 1 1" />
-            </geometry>
-            <material name="0.796078_0.823529_0.937255_0.000000_0.000000">
-                <color rgba="0.796078 0.823529 0.937255 1" />
-            </material>
-        </visual>
-    </link>
-    <link name="${prefix}gripper_block">
-        <inertial>
-            <mass value="1.56518e-06" />
-            <origin xyz="-0.005 0.0015 0.0075" rpy="0 -0 0" />
-            <inertia ixx="5.13549e-11" ixy="0" ixz="0" iyy="1.51997e-10" iyz="0" izz="1.0299e-10" />
-        </inertial>
-        <visual>
-            <origin xyz="-0.005 0.003 0.0075" rpy="0 -0 0" />
-            <geometry>
-                <mesh filename="package://gripper_description/meshes/soft-two-finger-gripper/Block.stl" scale="1 1 1" />
-            </geometry>
-            <material name="0.796078_0.823529_0.937255_0.000000_0.000000">
-                <color rgba="0.796078 0.823529 0.937255 1" />
-            </material>
-        </visual>
-    </link>
-    <link name="${prefix}gripper_block_1">
-        <inertial>
-            <mass value="1.56518e-06" />
-            <origin xyz="0.005 0.0015 0.0075" rpy="0 -0 0" />
-            <inertia ixx="5.13549e-11" ixy="0" ixz="0" iyy="1.51997e-10" iyz="0" izz="1.0299e-10" />
-        </inertial>
-        <visual>
-            <origin xyz="0.005 0.003 0.0075" rpy="0 -0 0" />
-            <geometry>
-                <mesh filename="package://gripper_description/meshes/soft-two-finger-gripper/Block.stl" scale="1 1 1" />
-            </geometry>
-            <material name="0.796078_0.823529_0.937255_0.000000_0.000000">
-                <color rgba="0.796078 0.823529 0.937255 1" />
-            </material>
-        </visual>
-    </link>
-    <link name="${prefix}gripper_block_2">
-        <inertial>
-            <mass value="1.56518e-06" />
-            <origin xyz="-0.005 0.0015 -0.0075" rpy="0 -0 0" />
-            <inertia ixx="5.13549e-11" ixy="0" ixz="0" iyy="1.51997e-10" iyz="0" izz="1.0299e-10" />
-        </inertial>
-        <visual>
-            <origin xyz="-0.005 0.003 -0.0075" rpy="0 -0 0" />
-            <geometry>
-                <mesh filename="package://gripper_description/meshes/soft-two-finger-gripper/Block.stl" scale="1 1 1" />
-            </geometry>
-            <material name="0.796078_0.823529_0.937255_0.000000_0.000000">
-                <color rgba="0.796078 0.823529 0.937255 1" />
-            </material>
-        </visual>
-    </link>
-    <link name="${prefix}gripper_block_3">
-        <inertial>
-            <mass value="1.56518e-06" />
-            <origin xyz="0.005 0.0015 -0.0075" rpy="0 -0 0" />
-            <inertia ixx="5.13549e-11" ixy="0" ixz="0" iyy="1.51997e-10" iyz="0" izz="1.0299e-10" />
-        </inertial>
-        <visual>
-            <origin xyz="0.005 0.003 -0.0075" rpy="0 -0 0" />
-            <geometry>
-                <mesh filename="package://gripper_description/meshes/soft-two-finger-gripper/Block.stl" scale="1 1 1" />
-            </geometry>
-            <material name="0.796078_0.823529_0.937255_0.000000_0.000000">
-                <color rgba="0.796078 0.823529 0.937255 1" />
-            </material>
-        </visual>
-    </link>
-    <link name="${prefix}gripper_clamp">
-        <inertial>
-            <mass value="2.4104e-05" />
-            <origin xyz="2.35624e-13 -5.97063e-12 0.018844" rpy="0 -0 0" />
-            <inertia ixx="1.14843e-08" ixy="0" ixz="0" iyy="2.35513e-08" iyz="0" izz="1.95862e-08" />
-        </inertial>
-        <visual>
-            <origin xyz="-0.0275 -3.46945e-18 0.005" rpy="0 -0 0" />
-            <geometry>
-                <mesh filename="package://gripper_description/meshes/soft-two-finger-gripper/Clamp.stl" scale="1 1 1" />
-            </geometry>
-            <material name="0.796078_0.823529_0.937255_0.000000_0.000000">
-                <color rgba="0.796078 0.823529 0.937255 1" />
-            </material>
-        </visual>
-    </link>
-    <link name="${prefix}gripper_dynamixel_xm430_w350_r">
-        <inertial>
-            <mass value="4.41073e-05" />
-            <origin xyz="-0.0166389 -0.00539576 -0.0143" rpy="0 -0 0" />
-            <inertia ixx="7.26484e-09" ixy="1.25677e-10" ixz="0" iyy="1.08932e-08" iyz="0" izz="1.24382e-08" />
-        </inertial>
-        <visual>
-            <origin xyz="-0.0396 0.011 -0.0286" rpy="0 -0 0" />
-            <geometry>
-                <mesh filename="package://gripper_description/meshes/soft-two-finger-gripper/dynamixel_XM430_W350_R.stl" scale="1 1 1" />
-            </geometry>
-            <material name="0.501961_0.501961_0.501961_0.000000_0.000000">
-                <color rgba="0.501961 0.501961 0.501961 1" />
-            </material>
-        </visual>
-    </link>
-    <link name="${prefix}gripper_gipper_case">
-        <inertial>
-            <mass value="2.86395e-05" />
-            <origin xyz="0.0180537 -0.0152097 -0.0161438" rpy="0 -0 0" />
-            <inertia ixx="1.17204e-08" ixy="-4.70838e-13" ixz="1.22897e-09" iyy="9.20144e-09" iyz="-3.20141e-12" izz="8.16469e-09" />
-        </inertial>
-        <visual>
-            <origin xyz="-0.006 -0.0152 0.0847" rpy="0 -0 0" />
-            <geometry>
-                <mesh filename="package://gripper_description/meshes/soft-two-finger-gripper/Gipper_case.stl" scale="1 1 1" />
-            </geometry>
-            <material name="1.000000_1.000000_1.000000_0.000000_0.000000">
-                <color rgba="1 1 1 1" />
-            </material>
-        </visual>
-    </link>
-    <link name="${prefix}gripper_gipper_case_1">
-        <inertial>
-            <mass value="2.86395e-05" />
-            <origin xyz="0.0180537 -0.0152097 -0.0161438" rpy="0 -0 0" />
-            <inertia ixx="1.17204e-08" ixy="-4.70838e-13" ixz="1.22897e-09" iyy="9.20144e-09" iyz="-3.20141e-12" izz="8.16469e-09" />
-        </inertial>
-        <visual>
-            <origin xyz="-0.006 -0.0152 0.0847" rpy="0 -0 0" />
-            <geometry>
-                <mesh filename="package://gripper_description/meshes/soft-two-finger-gripper/Gipper_case.stl" scale="1 1 1" />
-            </geometry>
-            <material name="1.000000_1.000000_1.000000_0.000000_0.000000">
-                <color rgba="1 1 1 1" />
-            </material>
-        </visual>
-    </link>
-    <link name="${prefix}gripper_gripper_support">
-        <inertial>
-            <mass value="1.89595e-05" />
-            <origin xyz="-0.00581655 -0.0152972 0.013" rpy="0 -0 0" />
-            <inertia ixx="3.98339e-09" ixy="2.93394e-10" ixz="0" iyy="3.42247e-09" iyz="1.43098e-15" izz="2.29475e-09" />
-        </inertial>
-        <visual>
-            <origin xyz="-0.0216198 -0.007 -0.0155" rpy="0 -0 0" />
-            <geometry>
-                <mesh filename="package://gripper_description/meshes/soft-two-finger-gripper/Gripper_support.stl" scale="1 1 1" />
-            </geometry>
-            <material name="1.000000_0.501961_0.501961_0.000000_0.000000">
-                <color rgba="1 0.501961 0.501961 1" />
-            </material>
-        </visual>
-    </link>
-    <link name="${prefix}gripper_gripper_support_1">
-        <inertial>
-            <mass value="1.89595e-05" />
-            <origin xyz="0.00230328 -0.0141822 0.01" rpy="0 -0 0" />
-            <inertia ixx="3.98339e-09" ixy="2.93394e-10" ixz="0" iyy="3.42247e-09" iyz="1.43098e-15" izz="2.29475e-09" />
-        </inertial>
-        <visual>
-            <origin xyz="-0.0135 -0.00588499 -0.0155" rpy="0 -0 0" />
-            <geometry>
-                <mesh filename="package://gripper_description/meshes/soft-two-finger-gripper/Gripper_support.stl" scale="1 1 1" />
-            </geometry>
-            <material name="1.000000_0.501961_0.501961_0.000000_0.000000">
-                <color rgba="1 0.501961 0.501961 1" />
-            </material>
-        </visual>
-    </link>
-    <link name="${prefix}gripper_link">
-        <inertial>
-            <mass value="3.47229e-06" />
-            <origin xyz="-0.0214556 -0.00340137 -0.00312234" rpy="0 -0 0" />
-            <inertia ixx="1.05957e-10" ixy="-3.94569e-11" ixz="3.16674e-11" iyy="7.05198e-10" iyz="6.17955e-12" izz="6.38214e-10" />
-        </inertial>
-        <visual>
-            <origin xyz="-0.035 0 0" rpy="0 -0 0" />
-            <geometry>
-                <mesh filename="package://gripper_description/meshes/soft-two-finger-gripper/Link.stl" scale="1 1 1" />
-            </geometry>
-            <material name="0.796078_0.823529_0.937255_0.000000_0.000000">
-                <color rgba="0.796078 0.823529 0.937255 1" />
-            </material>
-        </visual>
-    </link>
-    <link name="${prefix}gripper_link_1">
-        <inertial>
-            <mass value="3.47229e-06" />
-            <origin xyz="-0.0214556 -0.00340137 -0.00312234" rpy="0 -0 0" />
-            <inertia ixx="1.05957e-10" ixy="-3.94569e-11" ixz="3.16674e-11" iyy="7.05198e-10" iyz="6.17955e-12" izz="6.38214e-10" />
-        </inertial>
-        <visual>
-            <origin xyz="-0.035 0 0" rpy="0 -0 0" />
-            <geometry>
-                <mesh filename="package://gripper_description/meshes/soft-two-finger-gripper/Link.stl" scale="1 1 1" />
-            </geometry>
-            <material name="0.796078_0.823529_0.937255_0.000000_0.000000">
-                <color rgba="0.796078 0.823529 0.937255 1" />
-            </material>
-        </visual>
-    </link>
-    <link name="${prefix}gripper_link__1__loop_closure">
-        <inertial>
-            <mass value="1e-09" />
-            <origin xyz="0 0 0" rpy="0 -0 0" />
-            <inertia ixx="4e-14" ixy="0" ixz="0" iyy="4e-14" iyz="0" izz="4e-14" />
-        </inertial>
-    </link>
-    <link name="${prefix}gripper_link__2__loop_closure">
-        <inertial>
-            <mass value="1e-09" />
-            <origin xyz="0 0 0" rpy="0 -0 0" />
-            <inertia ixx="4e-14" ixy="0" ixz="0" iyy="4e-14" iyz="0" izz="4e-14" />
-        </inertial>
-    </link>
-    <link name="${prefix}gripper_mgnr09r315hm">
-        <inertial>
-            <mass value="7.10975e-06" />
-            <origin xyz="0.07 -0.00307814 -5.52605e-06" rpy="0 -0 0" />
-            <inertia ixx="7.3598e-11" ixy="0" ixz="0" iyy="1.27398e-08" iyz="1.15967e-13" izz="1.27163e-08" />
-        </inertial>
-        <visual>
-            <origin xyz="-0.0075 0 0.0045" rpy="0 -0 0" />
-            <geometry>
-                <mesh filename="package://gripper_description/meshes/soft-two-finger-gripper/MGNR09R315HM.stl" scale="1 1 1" />
-            </geometry>
-            <material name="0.796078_0.796078_0.796078_0.000000_0.000000">
-                <color rgba="0.796078 0.796078 0.796078 1" />
-            </material>
-        </visual>
-    </link>
-    <link name="${prefix}gripper_mgnr09r315hm_1">
-        <inertial>
-            <mass value="7.10975e-06" />
-            <origin xyz="0.07 -0.00307814 -5.52605e-06" rpy="0 -0 0" />
-            <inertia ixx="7.3598e-11" ixy="0" ixz="0" iyy="1.27398e-08" iyz="1.15967e-13" izz="1.27163e-08" />
-        </inertial>
-        <visual>
-            <origin xyz="-0.0075 0 0.0045" rpy="0 -0 0" />
-            <geometry>
-                <mesh filename="package://gripper_description/meshes/soft-two-finger-gripper/MGNR09R315HM.stl" scale="1 1 1" />
-            </geometry>
-            <material name="0.796078_0.796078_0.796078_0.000000_0.000000">
-                <color rgba="0.796078 0.796078 0.796078 1" />
-            </material>
-        </visual>
-    </link>
-    <link name="${prefix}gripper_planar_4" />
-    <link name="${prefix}gripper_planar_4_1" />
-    <link name="${prefix}gripper_planar_5" />
-    <link name="${prefix}gripper_planar_5_1" />
-    <link name="${prefix}gripper_root" />
-    <link name="${prefix}gripper_small_motor_mount">
-        <inertial>
-            <mass value="1.0786e-05" />
-            <origin xyz="0.000264358 -0.00445466 0.000270164" rpy="0 -0 0" />
-            <inertia ixx="7.45917e-10" ixy="1.29287e-13" ixz="-4.93148e-10" iyy="3.5822e-09" iyz="1.32127e-13" izz="2.98218e-09" />
-        </inertial>
-        <visual>
-            <origin xyz="0 0 0" rpy="0 -0 0" />
-            <geometry>
-                <mesh filename="package://gripper_description/meshes/soft-two-finger-gripper/Small_motor_mount.stl" scale="1 1 1" />
-            </geometry>
-            <material name="0.796078_0.823529_0.937255_0.000000_0.000000">
-                <color rgba="0.796078 0.823529 0.937255 1" />
-            </material>
-        </visual>
-    </link>
-    <link name="${prefix}gripper_small_motor_test_2_base">
-        <inertial>
-            <mass value="4.70869e-05" />
-            <origin xyz="-0.076 -0.023021 0.021" rpy="0 -0 0" />
-            <inertia ixx="1.97752e-08" ixy="0" ixz="0" iyy="1.84606e-07" iyz="0" izz="1.73024e-07" />
-        </inertial>
-        <visual>
-            <origin xyz="-0.156 -0.026 -0.004" rpy="0 -0 0" />
-            <geometry>
-                <mesh filename="package://gripper_description/meshes/soft-two-finger-gripper/Small_Motor_test_2_Base.stl" scale="1 1 1" />
-            </geometry>
-            <material name="0.000000_0.752941_0.752941_0.000000_0.000000">
-                <color rgba="0 0.752941 0.752941 1" />
-            </material>
-        </visual>
-    </link>
-    <link name="${prefix}gripper_soft_gripper_finger">
-        <inertial>
-            <mass value="4.70738e-05" />
-            <origin xyz="-0.0173609 0.0381915 -0.0129" rpy="0 -0 0" />
-            <inertia ixx="5.05765e-08" ixy="5.83018e-09" ixz="0" iyy="9.02641e-09" iyz="0" izz="5.43806e-08" />
-        </inertial>
-        <visual>
-            <origin xyz="-0.035 -0.005 0" rpy="0 -0 0" />
-            <geometry>
-                <mesh filename="package://gripper_description/meshes/soft-two-finger-gripper/soft_gripper_finger.stl" scale="1 1 1" />
-            </geometry>
-            <material name="0.231373_0.380392_0.705882_0.000000_0.000000">
-                <color rgba="0.231373 0.380392 0.705882 1" />
-            </material>
-        </visual>
-    </link>
-    <link name="${prefix}gripper_soft_gripper_finger_1">
-        <inertial>
-            <mass value="4.70738e-05" />
-            <origin xyz="-0.0173609 0.0381915 -0.0129" rpy="0 -0 0" />
-            <inertia ixx="5.05765e-08" ixy="5.83018e-09" ixz="0" iyy="9.02641e-09" iyz="0" izz="5.43806e-08" />
-        </inertial>
-        <visual>
-            <origin xyz="-0.035 -0.005 0" rpy="0 -0 0" />
-            <geometry>
-                <mesh filename="package://gripper_description/meshes/soft-two-finger-gripper/soft_gripper_finger.stl" scale="1 1 1" />
-            </geometry>
-            <material name="0.231373_0.380392_0.705882_0.000000_0.000000">
-                <color rgba="0.231373 0.380392 0.705882 1" />
-            </material>
-        </visual>
-    </link>
-    <joint name="${prefix}gripper_fastened_1" type="fixed">
-        <origin xyz="3.46945e-18 6.93889e-18 4.33681e-18" rpy="2.13568e-32 5.31737e-33 -1.5708" />
-        <axis xyz="0 0 1" />
-        <parent link="${prefix}gripper_root" />
-        <child link="${prefix}gripper_clamp" />
-    </joint>
-    <joint name="${prefix}gripper_fastened_10" type="fixed">
-        <origin xyz="0.0085 -0.018885 0.0282" rpy="1.5708 -8.04912e-16 3.14159" />
-        <axis xyz="0 -1 0" />
-        <parent link="${prefix}gripper_gripper_support_1" />
-        <child link="${prefix}gripper_gipper_case_1" />
-    </joint>
-    <joint name="${prefix}gripper_fastened_11" type="fixed">
-        <origin xyz="0.0858995 0.0065 0.0273995" rpy="-1.5708 -3.37038e-32 -1.3886e-31" />
-        <axis xyz="0 -1 0" />
-        <parent link="${prefix}gripper_base" />
-        <child link="${prefix}gripper_small_motor_test_2_base" />
-    </joint>
-    <joint name="${prefix}gripper_fastened_12" type="fixed">
-        <origin xyz="-0.0182005 0.04185 0.0213995" rpy="1.5708 -3.38813e-21 3.14159" />
-        <axis xyz="0 0 1" />
-        <parent link="${prefix}gripper_base" />
-        <child link="${prefix}gripper_dynamixel_xm430_w350_r" />
-    </joint>
-    <joint name="${prefix}gripper_fastened_13" type="fixed">
-        <origin xyz="0.0289911 -0.0021 -0.0217317" rpy="-1.5708 2.46733e-30 -3.29899e-29" />
-        <axis xyz="0 0 -1" />
-        <parent link="${prefix}gripper_gipper_case_1" />
-        <child link="${prefix}gripper_soft_gripper_finger" />
-    </joint>
-    <joint name="${prefix}gripper_fastened_14" type="fixed">
-        <origin xyz="0.0289911 -0.0021 -0.0217317" rpy="-1.5708 -7.02888e-17 -7.02888e-17" />
-        <axis xyz="0 0 1" />
-        <parent link="${prefix}gripper_gipper_case" />
-        <child link="${prefix}gripper_soft_gripper_finger_1" />
-    </joint>
-    <joint name="${prefix}gripper_fastened_2" type="fixed">
-        <origin xyz="0.0275 -0.00989949 0.027421" rpy="-1.44607e-16 -2.00374e-16 1.5708" />
-        <axis xyz="1.73472e-16 -1 -2.00618e-32" />
-        <parent link="${prefix}gripper_clamp" />
-        <child link="${prefix}gripper_base" />
-    </joint>
-    <joint name="${prefix}gripper_fastened_3" type="fixed">
-        <origin xyz="-0.0131198 -0.007 -0.0121" rpy="4.74207e-19 -1.38778e-16 -4.80745e-31" />
-        <axis xyz="0 -1 0" />
-        <parent link="${prefix}gripper_gripper_support" />
-        <child link="${prefix}gripper_block_1" />
-    </joint>
-    <joint name="${prefix}gripper_fastened_4" type="fixed">
-        <origin xyz="-0.0131198 -0.007 0.0381" rpy="6.13299e-17 -2.498e-16 -5.19187e-31" />
-        <axis xyz="0 -1 0" />
-        <parent link="${prefix}gripper_gripper_support" />
-        <child link="${prefix}gripper_block_3" />
-    </joint>
-    <joint name="${prefix}gripper_fastened_5" type="fixed">
-        <origin xyz="-0.005 -0.00588499 -0.0121" rpy="3.14159 -1.38778e-16 -3.14159" />
-        <axis xyz="0 -1 0" />
-        <parent link="${prefix}gripper_gripper_support_1" />
-        <child link="${prefix}gripper_block_2" />
-    </joint>
-    <joint name="${prefix}gripper_fastened_6" type="fixed">
-        <origin xyz="-0.146 -0.031 0.0035" rpy="-8.29972e-17 2.77556e-17 2.75156e-17" />
-        <axis xyz="0 1 0" />
-        <parent link="${prefix}gripper_small_motor_test_2_base" />
-        <child link="${prefix}gripper_mgnr09r315hm_1" />
-    </joint>
-    <joint name="${prefix}gripper_fastened_7" type="fixed">
-        <origin xyz="-0.146 -0.031 0.0385" rpy="-1.50861e-16 -2.498e-16 -1.44023e-16" />
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
Commit message: added tcp and tooltip tf

File: gripper_description/xacro/two-finger-gripper.urdf.xacro (robot description, xacro)
@@ -248,4 +248,6 @@
         </link>
         <link name="${prefix}gripper_root" />
+        <link name="${prefix}tcp" />
+        <link name="${prefix}tool_tip" />
         <link name="${prefix}gripper_small_motor_mount">
             <inertial>
@@ -317,4 +319,14 @@
             <parent link="${prefix}gripper_root" />
             <child link="${prefix}gripper_clamp" />
+        </joint>
+        <joint name="${prefix}tcp_joint" type="fixed">
+            <origin xyz="0 0 0.205" rpy="0 0 0" />
+            <parent link="${prefix}gripper_root" />
+            <child link="${prefix}tcp" />
+        </joint>
+        <joint name="${prefix}tool_tip_joint" type="fixed">
+            <origin xyz="0 0 0.25" rpy="0 0 0" />
+            <parent link="${prefix}gripper_root" />
+            <child link="${prefix}tool_tip" />
         </joint>
         <joint name="${prefix}gripper_fastened_2" type="fixed">
