Commit message: added collision boxes

File: gripper_description/xacro/two-finger-gripper.urdf.xacro (robot description, xacro)
@@ -22,4 +22,10 @@
                 </material>
             </visual>
+            <collision>
+                <origin xyz="-0.0701005 0.0525 0.0273995" rpy="0 -0 0" />
+                <geometry>
+                    <mesh filename="package://gripper_description/meshes/soft-two-finger-gripper/Base.stl" scale="1 1 1" />
+                </geometry>
+            </collision>
         </link>
         <link name="${prefix}gripper_block">
@@ -38,4 +44,10 @@
                 </material>
             </visual>
+            <collision>
+                <origin xyz="-0.005 0.003 0.0075" rpy="0 -0 0" />
+                <geometry>
+                    <mesh filename="package://gripper_description/meshes/soft-two-finger-gripper/Block.stl" scale="1 1 1" />
+                </geometry>
+            </collision>
         </link>
         <link name="${prefix}gripper_block_1">
@@ -54,4 +66,10 @@
                 </material>
             </visual>
+            <collision>
+                <origin xyz="-0.01375 0.0015 0" rpy="0 -0 0" />
+                <geometry>
+                    <mesh filename="package://gripper_description/meshes/soft-two-finger-gripper/Block.stl" scale="1 1 1" />
+                </geometry>
+            </collision>
         </link>
         <link name="${prefix}gripper_block_2">
@@ -70,4 +88,10 @@
                 </material>
             </visual>
+            <collision>
+                <origin xyz="0.01375 0.0015 0" rpy="0 -0 0" />
+                <geometry>
+                    <mesh filename="package://gripper_description/meshes/soft-two-finger-gripper/Block.stl" scale="1 1 1" />
+                </geometry>
+            </collision>
         </link>
         <link name="${prefix}gripper_block_3">
@@ -86,4 +110,10 @@
                 </material>
             </visual>
+            <collision>
+                <origin xyz="0.005 0.003 -0.0075" rpy="0 -0 0" />
+                <geometry>
+                    <mesh filename="package://gripper_description/meshes/soft-two-finger-gripper/Block.stl" scale="1 1 1" />
+                </geometry>
+            </collision>
         </link>
         <link name="${prefix}gripper_clamp">
@@ -102,4 +132,10 @@
                 </material>
             </visual>
+            <collision>
+                <origin xyz="-0.0275 -3.46945e-18 0.005" rpy="0 -0 0" />
+                <geometry>
+                    <mesh filename="package://gripper_description/meshes/soft-two-finger-gripper/Clamp.stl" scale="1 1 1" />
+                </geometry>
+            </collision>
         </link>
         <link name="${prefix}gripper_dynamixel_xm430_w350_r">
@@ -118,4 +154,10 @@
                 </material>
             </visual>
+            <collision>
+                <origin xyz="-0.0396 0.011 -0.0286" rpy="0 -0 0" />
+                <geometry>
+                    <mesh filename="package://gripper_description/meshes/soft-two-finger-gripper/dynamixel_XM430_W350_R.stl" scale="1 1 1" />
+                </geometry>
+            </collision>
         </link>
         <link name="${prefix}gripper_gipper_case">
@@ -134,4 +176,10 @@
                 </material>
             </visual>
+            <collision>
+                <origin xyz="-0.006 -0.0152 0.0847" rpy="0 -0 0" />
+                <geometry>
+                    <mesh filename="package://gripper_description/meshes/soft-two-finger-gripper/Gipper_case.stl" scale="1 1 1" />
+                </geometry>
+            </collision>
         </link>
         <link name="${prefix}gripper_gipper_case_1">
@@ -150,4 +198,10 @@
                 </material>
             </visual>
+            <collision>
+                <origin xyz="-0.006 -0.0152 0.0847" rpy="0 -0 0" />
+                <geometry>
+                    <mesh filename="package://gripper_description/meshes/soft-two-finger-gripper/Gipper_case.stl" scale="1 1 1" />
+                </geometry>
+            </collision>
         </link>
         <link name="${prefix}gripper_gripper_support">
@@ -166,4 +220,10 @@
                 </material>
             </visual>
+            <collision>
+                <origin xyz="-0.0085 0 -0.0034" rpy="0 -0 0" />
+                <geometry>
+                    <mesh filename="package://gripper_description/meshes/soft-two-finger-gripper/Gripper_support.stl" scale="1 1 1" />
+                </geometry>
+            </collision>
         </link>
         <link name="${prefix}gripper_gripper_support_1">
@@ -182,4 +242,10 @@
                 </material>
             </visual>
+            <collision>
+                <origin xyz="-0.0085 0 -0.0034" rpy="0 -0 0" />
+                <geometry>
+                    <mesh filename="package://gripper_description/meshes/soft-two-finger-gripper/Gripper_support.stl" scale="1 1 1" />
+                </geometry>
+            </collision>
         </link>
         <link name="${prefix}gripper_link">
@@ -198,4 +264,10 @@
                 </material>
             </visual>
+            <collision>
+                <origin xyz="-0.035 0 0" rpy="0 -0 0" />
+                <geometry>
+                    <mesh filename="package://gripper_description/meshes/soft-two-finger-gripper/Link.stl" scale="1 1 1" />
+                </geometry>
+            </collision>
         </link>
         <link name="${prefix}gripper_link_1">
@@ -214,4 +286,10 @@
                 </material>
             </visual>
+            <collision>
+                <origin xyz="-0.035 0 0" rpy="0 -0 0" />
+                <geometry>
+                    <mesh filename="package://gripper_description/meshes/soft-two-finger-gripper/Link.stl" scale="1 1 1" />
+                </geometry>
+            </collision>
         </link>
         <link name="${prefix}gripper_mgnr09r315hm">
@@ -230,4 +308,10 @@
                 </material>
             </visual>
+            <collision>
+                <origin xyz="-0.0075 0 0.0045" rpy="0 -0 0" />
+                <geometry>
+                    <mesh filename="package://gripper_description/meshes/soft-two-finger-gripper/MGNR09R315HM.stl" scale="1 1 1" />
+                </geometry>
+            </collision>
         </link>
         <link name="${prefix}gripper_mgnr09r315hm_1">
@@ -246,4 +330,10 @@
                 </material>
             </visual>
+            <collision>
+                <origin xyz="-0.0075 0 0.0045" rpy="0 -0 0" />
+                <geometry>
+                    <mesh filename="package://gripper_description/meshes/soft-two-finger-gripper/MGNR09R315HM.stl" scale="1 1 1" />
+                </geometry>
+            </collision>
         </link>
         <link name="${prefix}gripper_root" />
@@ -265,4 +355,10 @@
                 </material>
             </visual>
+            <collision>
+                <origin xyz="0 0 0" rpy="0 -0 0" />
+                <geometry>
+                    <mesh filename="package://gripper_description/meshes/soft-two-finger-gripper/Small_motor_mount.stl" scale="1 1 1" />
+                </geometry>
+            </collision>
         </link>
         <link name="${prefix}gripper_small_motor_test_2_base">
@@ -281,4 +377,10 @@
                 </material>
             </visual>
+            <collision>
+                <origin xyz="-0.156 -0.026 -0.004" rpy="0 -0 0" />
+                <geometry>
+                    <mesh filename="package://gripper_description/meshes/soft-two-finger-gripper/Small_Motor_test_2_Base.stl" scale="1 1 1" />
+                </geometry>
+            </collision>
         </link>
         <link name="${prefix}gripper_soft_gripper_finger">
@@ -297,4 +399,10 @@
                 </material>
             </visual>
+            <collision>
+                <origin xyz="-0.035 -0.005 0" rpy="0 -0 0" />
+                <geometry>
+                    <mesh filename="package://gripper_description/meshes/soft-two-finger-gripper/soft_gripper_finger.stl" scale="1 1 1" />
+                </geometry>
+            </collision>
         </link>
         <link name="${prefix}gripper_soft_gripper_finger_1">
@@ -313,4 +421,10 @@
                 </material>
             </visual>
+            <collision>
+                <origin xyz="-0.035 -0.005 0" rpy="0 -0 0" />
+                <geometry>
+                    <mesh filename="package://gripper_description/meshes/soft-two-finger-gripper/soft_gripper_finger.stl" scale="1 1 1" />
+                </geometry>
+            </collision>
         </link>
         <joint name="${prefix}gripper_fastened_1" type="fixed">
