Commit message: updated tcp and refactored estimation nodes into a new package

File: gripper_description/xacro/two-finger-gripper.urdf.xacro (robot description, xacro)
@@ -434,6 +434,8 @@
             <child link="${prefix}gripper_clamp" />
         </joint>
+        <!-- from gripper_root to the finger base is 125mm -->
+        <!-- from finger base to the tcp 62mm -->
         <joint name="${prefix}tcp_joint" type="fixed">
-            <origin xyz="0 0 0.205" rpy="0 0 0" />
+            <origin xyz="0 0 0.187" rpy="0 0 0" />
             <parent link="${prefix}gripper_root" />
             <child link="${prefix}tcp" />
